File: 1. PCB/GBA Wireless Gamepad.brd (EAGLE design)
At the start: 39.9 x 26.7 mm, 14 parts, among them J1 UART-CP2102, J3 GBA EXT, U1 ESP-WROOM-32

Commit message: no message
Parts:
- U$10: device ,giltesa_logos:GILTESA.COM_MASK -> ,giltesa_logos:GILTESA.COM_MASK_15MM
Other:
- board text removed: "JLCJLCJLCJLC"
Changed lines of the file:
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@@
 <layer number="16" name="Bottom" color="1" fill="1" visible="yes" active="yes"/>
 <layer number="17" name="Pads" color="2" fill="1" visible="yes" active="yes"/>
-<layer number="18" name="Vias" color="2" fill="1" visible="yes" active="yes"/>
+<layer number="18" name="Vias" color="14" fill="1" visible="yes" active="yes"/>
 <layer number="19" name="Unrouted" color="6" fill="1" visible="yes" active="yes"/>
 <layer number="20" name="Dimension" color="15" fill="1" visible="yes" active="yes"/>
@@
 <layer number="154" name="FabDoc2" color="2" fill="1" visible="no" active="no"/>
 <layer number="155" name="FabDoc3" color="7" fill="15" visible="no" active="no"/>
+<layer number="156" name="DXF0409-TOP" color="7" fill="1" visible="no" active="no"/>
+<layer number="157" name="DXF0409-BOTTOM" color="7" fill="1" visible="no" active="no"/>
+<layer number="158" name="FaceMMeas" color="7" fill="1" visible="no" active="no"/>
+<layer number="159" name="Geh-Bear2" color="7" fill="1" visible="no" active="no"/>
+<layer number="160" name="Topologie" color="7" fill="1" visible="no" active="no"/>
+<layer number="161" name="tomplace2" color="7" fill="1" visible="no" active="no"/>
+<layer number="162" name="RemovedThings" color="12" fill="11" visible="yes" active="yes"/>
+<layer number="166" name="AntennaArea" color="7" fill="1" visible="no" active="no"/>
+<layer number="168" name="4mmHeightArea" color="7" fill="1" visible="no" active="no"/>
 <layer number="188" name="Graphics" color="15" fill="1" visible="no" active="yes"/>
 <layer number="191" name="mNets" color="7" fill="1" visible="no" active="yes"/>
@@
 <layer number="250" name="Descript" color="3" fill="1" visible="no" active="no"/>
 <layer number="251" name="SMDround" color="12" fill="11" visible="no" active="no"/>
+<layer number="252" name="BR-BS" color="7" fill="1" visible="no" active="no"/>
+<layer number="253" name="Extra" color="7" fill="1" visible="no" active="no"/>
 <layer number="254" name="cooling" color="7" fill="1" visible="no" active="yes"/>
 <layer number="255" name="HELP" color="7" fill="1" visible="no" active="yes"/>
@@
 <wire x1="0" y1="12.573" x2="0" y2="0" width="0.254" layer="20"/>
 <text x="19.431" y="21.082" size="1.27" layer="22" font="vector" ratio="16" rot="MR0" align="center">GBA BLUETOOTH GAMEPAD</text>
-<text x="25.527" y="2.54" size="0.9144" layer="21" align="center">JLCJLCJLCJLC</text>
 </plain>
 <attributes>
@@
 <element name="U$14" library="SparkFun" package="FIDUCIAL-1X2" value="FIDUCIAL1X2" x="7.874" y="9.398" smashed="yes"/>
 <element name="U$17" library="cc-by-nc-sa" package="CC-NC-B_NIX" value="CC-NC-BCNIX" x="-0.127" y="0" smashed="yes"/>
-<element name="U$10" library=",giltesa_logos" package="GILTESA.COM_MASK" value="GILTESA.COM_MASK" x="26.924" y="21.971" smashed="yes" rot="MR0"/>
+<element name="U$10" library=",giltesa_logos" package="GILTESA.COM_MASK_15MM" value="GILTESA.COM_MASK" x="26.924" y="21.971" smashed="yes" rot="MR0"/>
 <element name="LOGO1" library="ohw-logo" package="OSHW_FILLX150_NOTEXT" value="OSHW_LOGO_FILLX0150-NT" x="8.128" y="20.701" smashed="yes"/>
 <element name="U1" library=",giltesa" package="ESP32-WROOM-NARROW" value="ESP-WROOM-32" x="25.527" y="12.065" smashed="yes">
@@
 <wire x1="35.56" y1="18.034" x2="35.099" y2="18.495" width="0.4572" layer="1"/>
 <wire x1="33.765" y1="18.495" x2="35.099" y2="18.495" width="0.4572" layer="1"/>
-<via x="35.56" y="16.764" extent="1-16" drill="0.5588"/>
-<via x="36.576" y="16.764" extent="1-16" drill="0.5588"/>
-<via x="37.592" y="16.764" extent="1-16" drill="0.5588"/>
-<via x="1.905" y="5.334" extent="1-16" drill="0.5588"/>
-<via x="2.921" y="5.334" extent="1-16" drill="0.5588"/>
-<via x="3.937" y="5.334" extent="1-16" drill="0.5588"/>
+<via x="35.56" y="16.764" extent="1-16" drill="0.3048"/>
+<via x="36.576" y="16.764" extent="1-16" drill="0.3048"/>
+<via x="37.592" y="16.764" extent="1-16" drill="0.3048"/>
+<via x="1.905" y="5.334" extent="1-16" drill="0.3048"/>
+<via x="2.921" y="5.334" extent="1-16" drill="0.3048"/>
+<via x="3.937" y="5.334" extent="1-16" drill="0.3048"/>
 <wire x1="17.289" y1="18.495" x2="16.59" y2="18.495" width="0.4572" layer="1"/>
 <wire x1="16.59" y1="18.495" x2="14.859" y2="16.764" width="0.4572" layer="1"/>
 <wire x1="5.068" y1="18.034" x2="5.068" y2="17.157" width="0.4572" layer="1"/>
 <wire x1="35.56" y1="18.034" x2="35.56" y2="16.764" width="0.4572" layer="1"/>
-<via x="7.874" y="16.129" extent="1-16" drill="0.5588"/>
-<via x="24.257" y="15.113" extent="1-16" drill="0.5588"/>
-<via x="23.241" y="15.113" extent="1-16" drill="0.5588"/>
-<via x="25.273" y="15.113" extent="1-16" drill="0.5588"/>
-<via x="22.225" y="15.113" extent="1-16" drill="0.5588"/>
-<via x="21.209" y="15.113" extent="1-16" drill="0.5588"/>
-<via x="21.209" y="13.081" extent="1-16" drill="0.5588"/>
-<via x="21.209" y="12.065" extent="1-16" drill="0.5588"/>
-<via x="21.209" y="11.049" extent="1-16" drill="0.5588"/>
-<via x="21.209" y="14.097" extent="1-16" drill="0.5588"/>
-<via x="25.146" y="3.683" extent="1-16" drill="0.5588"/>
-<via x="26.162" y="3.683" extent="1-16" drill="0.5588"/>
-<via x="24.13" y="3.683" extent="1-16" drill="0.5588"/>
-<via x="27.178" y="3.683" extent="1-16" drill="0.5588"/>
-<via x="27.178" y="4.699" extent="1-16" drill="0.5588"/>
-<via x="28.194" y="4.699" extent="1-16" drill="0.5588"/>
-<via x="29.21" y="4.699" extent="1-16" drill="0.5588"/>
-<via x="24.13" y="4.699" extent="1-16" drill="0.5588"/>
-<via x="23.114" y="4.699" extent="1-16" drill="0.5588"/>
-<via x="22.098" y="4.699" extent="1-16" drill="0.5588"/>
-<via x="21.336" y="3.937" extent="1-16" drill="0.5588"/>
-<via x="29.972" y="3.937" extent="1-16" drill="0.5588"/>
-<via x="7.112" y="15.367" extent="1-16" drill="0.5588"/>
-<via x="8.636" y="15.367" extent="1-16" drill="0.5588"/>
-<via x="6.35" y="14.605" extent="1-16" drill="0.5588"/>
-<via x="7.874" y="14.605" extent="1-16" drill="0.5588"/>
-<via x="9.398" y="14.605" extent="1-16" drill="0.5588"/>
-<via x="5.588" y="13.589" extent="1-16" drill="0.5588"/>
-<via x="4.826" y="12.827" extent="1-16" drill="0.5588"/>
-<via x="6.35" y="12.827" extent="1-16" drill="0.5588"/>
-<via x="4.064" y="12.065" extent="1-16" drill="0.5588"/>
-<via x="5.588" y="12.065" extent="1-16" drill="0.5588"/>
-<via x="7.112" y="12.065" extent="1-16" drill="0.5588"/>
-<via x="10.16" y="13.589" extent="1-16" drill="0.5588"/>
-<via x="9.398" y="12.827" extent="1-16" drill="0.5588"/>
-<via x="10.922" y="12.827" extent="1-16" drill="0.5588"/>
-<via x="8.636" y="12.065" extent="1-16" drill="0.5588"/>
-<via x="10.16" y="12.065" extent="1-16" drill="0.5588"/>
-<via x="11.684" y="12.065" extent="1-16" drill="0.5588"/>
-<via x="2.921" y="6.35" extent="1-16" drill="0.5588"/>
-<via x="2.921" y="4.318" extent="1-16" drill="0.5588"/>
+<via x="7.874" y="16.129" extent="1-16" drill="0.3048"/>
+<via x="24.257" y="15.113" extent="1-16" drill="0.3048"/>
+<via x="23.241" y="15.113" extent="1-16" drill="0.3048"/>
+<via x="25.273" y="15.113" extent="1-16" drill="0.3048"/>
+<via x="22.225" y="15.113" extent="1-16" drill="0.3048"/>
+<via x="21.209" y="15.113" extent="1-16" drill="0.3048"/>
+<via x="21.209" y="13.081" extent="1-16" drill="0.3048"/>
+<via x="21.209" y="12.065" extent="1-16" drill="0.3048"/>
+<via x="21.209" y="11.049" extent="1-16" drill="0.3048"/>
+<via x="21.209" y="14.097" extent="1-16" drill="0.3048"/>
+<via x="25.146" y="3.683" extent="1-16" drill="0.3048"/>
+<via x="26.162" y="3.683" extent="1-16" drill="0.3048"/>
+<via x="24.13" y="3.683" extent="1-16" drill="0.3048"/>
+<via x="27.178" y="3.683" extent="1-16" drill="0.3048"/>
+<via x="27.178" y="4.699" extent="1-16" drill="0.3048"/>
+<via x="28.194" y="4.699" extent="1-16" drill="0.3048"/>
+<via x="29.21" y="4.699" extent="1-16" drill="0.3048"/>
+<via x="24.13" y="4.699" extent="1-16" drill="0.3048"/>
+<via x="23.114" y="4.699" extent="1-16" drill="0.3048"/>
+<via x="22.098" y="4.699" extent="1-16" drill="0.3048"/>
+<via x="21.336" y="3.937" extent="1-16" drill="0.3048"/>
+<via x="29.972" y="3.937" extent="1-16" drill="0.3048"/>
+<via x="7.112" y="15.367" extent="1-16" drill="0.3048"/>
+<via x="8.636" y="15.367" extent="1-16" drill="0.3048"/>
+<via x="6.35" y="14.605" extent="1-16" drill="0.3048"/>
+<via x="7.874" y="14.605" extent="1-16" drill="0.3048"/>
+<via x="9.398" y="14.605" extent="1-16" drill="0.3048"/>
+<via x="5.588" y="13.589" extent="1-16" drill="0.3048"/>
+<via x="4.826" y="12.827" extent="1-16" drill="0.3048"/>
+<via x="6.35" y="12.827" extent="1-16" drill="0.3048"/>
+<via x="4.064" y="12.065" extent="1-16" drill="0.3048"/>
+<via x="5.588" y="12.065" extent="1-16" drill="0.3048"/>
+<via x="7.112" y="12.065" extent="1-16" drill="0.3048"/>
+<via x="10.16" y="13.589" extent="1-16" drill="0.3048"/>
+<via x="9.398" y="12.827" extent="1-16" drill="0.3048"/>
+<via x="10.922" y="12.827" extent="1-16" drill="0.3048"/>
+<via x="8.636" y="12.065" extent="1-16" drill="0.3048"/>
+<via x="10.16" y="12.065" extent="1-16" drill="0.3048"/>
+<via x="11.684" y="12.065" extent="1-16" drill="0.3048"/>
+<via x="2.921" y="6.35" extent="1-16" drill="0.3048"/>
+<via x="2.921" y="4.318" extent="1-16" drill="0.3048"/>
 <contactref element="J3" pad="6"/>
 <contactref element="S1" pad="1"/>
